File: z80_cpm_mmu.sch (KiCad schematic (older format))
At the start: 17 parts, among them P1 BUS, P2 ROM, P3 OUT, P4 RAM, P5 AUX, P6 EXT, U1 74HCT04, U3 74LS32, U4 74HCT00

Commit message: Fix IC references to be contiguous
Parts:
- renumbered U4 to U2
Changed lines of the file:
@@
-EESchema Schematic File Version 2  date 13/06/2016 14:27:26
+EESchema Schematic File Version 2  date 13/06/2016 15:28:09
 LIBS:power
 LIBS:device
@@
 $EndComp
 $Comp
-L 74HCT00 U4
+L 74HCT00 U2
 U 3 1 575E8C9F
 P 4200 1600
-F 0 "U4" H 4200 1650 60  0000 C CNN
+F 0 "U2" H 4200 1650 60  0000 C CNN
 F 1 "74HCT00" H 4200 1500 60  0000 C CNN
 F 2 "~" H 4200 1600 60  0000 C CNN
@@
 	3700 2400 5300 2400
 $Comp
-L 74HCT00 U4
+L 74HCT00 U2
 U 1 1 575E94D3
 P 3100 3000
-F 0 "U4" H 3100 3050 60  0000 C CNN
+F 0 "U2" H 3100 3050 60  0000 C CNN
 F 1 "74HCT00" H 3100 2900 60  0000 C CNN
 F 2 "~" H 3100 3000 60  0000 C CNN
@@
 $EndComp
 $Comp
-L 74HCT00 U4
+L 74HCT00 U2
 U 2 1 575E94D9
 P 3100 3600
-F 0 "U4" H 3100 3650 60  0000 C CNN
+F 0 "U2" H 3100 3650 60  0000 C CNN
 F 1 "74HCT00" H 3100 3500 60  0000 C CNN
 F 2 "~" H 3100 3600 60  0000 C CNN
@@
 	5300 3300 5100 3300
 $Comp
-L 74HCT00 U4
+L 74HCT00 U2
 U 4 1 575E9604
 P 7000 2800
-F 0 "U4" H 7000 2850 60  0000 C CNN
+F 0 "U2" H 7000 2850 60  0000 C CNN
 F 1 "74HCT00" H 7000 2700 60  0000 C CNN
 F 2 "~" H 7000 2800 60  0000 C CNN
